File: kwatch-v1-rev1.sch (EAGLE design)
At the start: 2 parts, among them IC1 STM32F10XCXT6

Commit message: Updated - still in progress
Parts:
- added BM-S1: RF-BM-S02, szrfstar:RF-BM-S02
- added IC2: TP4056, TP4056:TP4056
- added R1: (no value), resistor:R-EU_R0805
- added U1: (no value), MicroUSB:USB""
- added U2: LP2985AIM5-3.3, LP2985AIM5X-3.3:LP2985AIM5-3.3
- renumbered JP1 to JP_OLED
Connections:
- new net CHRG: IC2.CHRG
- new net N$2: IC2.PROG, R1.2
- new net STDBY: IC2.STDBY
- new net USB+: IC2.CE, IC2.VCC, U1.VBUS
- new net VCC: BM-S1.VCC
- net BAT+: now also IC2.BAT
- net GND: now also BM-S1.EN(P2.0), BM-S1.GND, IC2.GND, IC2.TEMP, R1.1, U1.GND, U2.GND
- net USART1_RX: now also BM-S1.(P0.3)TX
- net USART1_TX: now also BM-S1.(P0.2)RX
